File: mega_shield_simple.brd (EAGLE design)
At the start: 101.6 x 53.3 mm, 24 parts, among them J2 Mega R3, M1_FUSE FUSELITTLEFUSE, M1_PWR 1X2-3.5MM, M2_FUSE FUSELITTLEFUSE, M2_PWR 1X2-3.5MM

Commit message: add fuses to sch and brd files
Parts:
- added 12V_FUSE: 3568, keystone:3568
- added 12V_PASS1, 12V_PASS2: 1X2-3.5MM, adafruit:1X2-3.5MM
- M1_FUSE, M2_FUSE: value FUSELITTLEFUSE -> FUSETE5; device fuse:LITTLEFUSE -> fuse:TE5
- moved M1_PWR 4.95 mm to (5.08, 10.2)
- moved 5V_OUT 4.78 mm to (5.08, 18.4)
- moved M2_PWR 4.78 mm to (5.08, 26.7)
- moved M2_FUSE 4.45 mm to (17.8, 23.9)
- moved R9 4.13 mm to (21.4, 37.3), turned to 90 degrees
- moved JP1 2.54 mm to (31.8, 19.4)
- moved JP2 2.54 mm to (31.8, 38.2)
- moved LED5 2.16 mm to (25.1, 43.7)
- moved M1_FUSE 0.25 mm to (17.8, 13.1)
Connections:
- new net 12V_PASSTHRU1: 12V_FUSE.1, 12V_FUSE.2, 12V_PASS2.1
- new net 12V_PASSTHRU2: 12V_FUSE.3, 12V_FUSE.4, 12V_PASS1.1
- net GND: now also 12V_PASS1.2, 12V_PASS2.2
Routing:
- net GND: track 246.0 -> 268.3 mm
- net 12V_PASSTHRU1: track 0.00 -> 11.5 mm
- net 12V_PASSTHRU2: track 0.00 -> 11.5 mm
- net M2_PWR1: track 7.82 -> 14.7 mm
- net M1_PWR2: track 24.7 -> 29.7 mm
- net M1_PWR1: track 6.89 -> 11.5 mm
- net M2_PWR2: track 24.7 -> 29.2 mm
- net N$9: track 7.63 -> 12.1 mm
- net MEGA2: track 63.1 -> 58.7 mm
- net MEGA3: track 58.6 -> 54.7 mm
- net N$7: track 8.17 -> 10.6 mm
- net RESET: track 15.7 -> 18.0 mm
- net MEGA19: track 60.6 -> 58.7 mm
- net MEGA_5V: track 159.0 -> 160.9 mm
- net MEGA18: track 55.7 -> 54.4 mm
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Other:
- board text added: "+12V"
- board text added: "Status"
- board text added: "We'll carry on"
