File: mega_shield_simple.sch (EAGLE design)
At the start: 24 parts, among them J2 Mega R3, M1_FUSE FUSELITTLEFUSE, M1_PWR 1X2-3.5MM, M2_FUSE FUSELITTLEFUSE, M2_PWR 1X2-3.5MM

Commit message: add fuses to sch and brd files
Parts:
- added 12V_FUSE: 3568, keystone:3568
- added 12V_PASS1, 12V_PASS2: 1X2-3.5MM, adafruit:1X2-3.5MM
- M1_FUSE, M2_FUSE: value FUSELITTLEFUSE -> FUSETE5; device fuse:FUSELITTLEFUSE -> fuse:FUSETE5
Connections:
- new net 12V_PASSTHRU1: 12V_FUSE.1, 12V_PASS2.1
- new net 12V_PASSTHRU2: 12V_FUSE.2, 12V_PASS1.1
- net GND: now also 12V_PASS1.2, 12V_PASS2.2
Other:
- note added: "12V pass through"
Changed lines of the file:
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@@
 <class number="0" name="default" width="0" drill="0">
 </class>
-<class number="1" name="12V_PWR" width="2.159" drill="0">
+<class number="1" name="12V_PWR" width="1.778" drill="0">
 </class>
 <class number="2" name="5V_LDO" width="0.3048" drill="0">
@@
 <part name="C9" library="rcl" deviceset="C-US" device="025-050X050" value="0.1 uF"/>
 <part name="GND21" library="supply1" deviceset="GND" device=""/>
-<part name="M1_FUSE" library="fuse" deviceset="FUSE" device="LITTLEFUSE" value="FUSELITTLEFUSE"/>
-<part name="M2_FUSE" library="fuse" deviceset="FUSE" device="LITTLEFUSE" value="FUSELITTLEFUSE"/>
+<part name="M1_FUSE" library="fuse" deviceset="FUSE" device="TE5" value="FUSETE5"/>
+<part name="M2_FUSE" library="fuse" deviceset="FUSE" device="TE5" value="FUSETE5"/>
 <part name="M2_PWR" library="adafruit" deviceset="1X2" device="-3.5MM"/>
 <part name="5V_OUT" library="adafruit" deviceset="1X2" device="-3.5MM"/>
 <part name="GND2" library="supply1" deviceset="GND" device=""/>
+<part name="12V_PASS2" library="adafruit" deviceset="1X2" device="-3.5MM"/>
+<part name="12V_PASS1" library="adafruit" deviceset="1X2" device="-3.5MM"/>
+<part name="12V_FUSE" library="keystone" deviceset="3568" device="" value="3568"/>
+<part name="GND4" library="supply1" deviceset="GND" device=""/>
 </parts>
 <sheets>
@@
 <text x="-5.08" y="-12.7" size="1.778" layer="91">These screw terminals connect each motor to the motor driver</text>
 <text x="-17.78" y="-68.58" size="1.778" layer="91">The motors connect to the above 6-pin headers</text>
+<text x="43.18" y="20.32" size="1.778" layer="91">12V pass through</text>
 </plain>
 <instances>
@@
 <instance part="5V_OUT" gate="G$1" x="-55.88" y="-33.02" rot="R90"/>
 <instance part="GND2" gate="1" x="-58.42" y="-40.64"/>
+<instance part="12V_PASS2" gate="G$1" x="45.72" y="12.7" rot="R90"/>
+<instance part="12V_PASS1" gate="G$1" x="66.04" y="12.7" rot="R90"/>
+<instance part="12V_FUSE" gate="G$1" x="43.18" y="0" smashed="yes" rot="R270">
+<attribute name="NAME" x="39.497" y="8.89" size="1.778" layer="95" rot="R270"/>
+</instance>
+<instance part="GND4" gate="1" x="71.12" y="-2.54"/>
 </instances>
 <busses>
@@
 <pinref part="GND2" gate="1" pin="GND"/>
 </segment>
+<segment>
+<pinref part="12V_PASS2" gate="G$1" pin="2"/>
+<wire x1="45.72" y1="7.62" x2="45.72" y2="0" width="0.1524" layer="91"/>
+<pinref part="12V_PASS1" gate="G$1" pin="2"/>
+<wire x1="45.72" y1="0" x2="66.04" y2="0" width="0.1524" layer="91"/>
+<wire x1="66.04" y1="0" x2="66.04" y2="7.62" width="0.1524" layer="91"/>
+<pinref part="GND4" gate="1" pin="GND"/>
+<wire x1="71.12" y1="0" x2="66.04" y2="0" width="0.1524" layer="91"/>
+<junction x="66.04" y="0"/>
+</segment>
 </net>
 <net name="MEGASDA" class="0">
@@
 </segment>
 </net>
+<net name="12V_PASSTHRU1" class="0">
+<segment>
+<pinref part="12V_PASS2" gate="G$1" pin="1"/>
+<pinref part="12V_FUSE" gate="G$1" pin="1"/>
+<wire x1="43.18" y1="5.08" x2="43.18" y2="7.62" width="0.1524" layer="91"/>
+</segment>
+</net>
+<net name="12V_PASSTHRU2" class="0">
+<segment>
+<pinref part="12V_PASS1" gate="G$1" pin="1"/>
+<wire x1="63.5" y1="7.62" x2="63.5" y2="-5.08" width="0.1524" layer="91"/>
+<pinref part="12V_FUSE" gate="G$1" pin="2"/>
+<wire x1="63.5" y1="-5.08" x2="43.18" y2="-5.08" width="0.1524" layer="91"/>
+</segment>
+</net>
